File: hardware/memory-core-prototype-a/03_CODEC_CONVERSION.kicad_sch (KiCad schematic)
At the start: 1 part, among them J903 SHEET_INTERFACE_NOT_FITTED

Commit message: Capture ERC-validated codec conversion sheet
Parts:
- removed J903: SHEET_INTERFACE_NOT_FITTED, symbol Connector_Generic:Conn_01x15
- added C300, C301: 10µF bulk, Capacitor_SMD:C_0805_2012Metric, symbol Device:C
- added C302, C303, C304, C305, C306, C307: 1µF local, Capacitor_SMD:C_0805_2012Metric, symbol Device:C
- added C308, C309, C310, C311: 10µF reference, Capacitor_SMD:C_0805_2012Metric, symbol Device:C
- added C312, C313, C314, C315, C316: 100nF unused ADC, Capacitor_SMD:C_0805_2012Metric, symbol Device:C
- added C320, C324: 100nF + rail, Capacitor_SMD:C_0805_2012Metric, symbol Device:C
- added C321, C325: 100nF - rail, Capacitor_SMD:C_0805_2012Metric, symbol Device:C
- added C322, C326: 4.7µF + rail, Capacitor_SMD:C_0805_2012Metric, symbol Device:C
- added C323, C327: 4.7µF - rail, Capacitor_SMD:C_0805_2012Metric, symbol Device:C
- added C330, C332: 1µF AC, symbol Device:C
- added C331, C333: 2.2nF anti-alias, Capacitor_SMD:C_0805_2012Metric, symbol Device:C
- added C340, C341, C345, C346, C350, C351: 10µF AC, symbol Device:C
- added C342, C347, C352: 3.3nF, Capacitor_SMD:C_0805_2012Metric, symbol Device:C
- added C343, C344, C348, C349, C353, C354: 680pF, Capacitor_SMD:C_0805_2012Metric, symbol Device:C
- added D300, D301: BAT54-class, symbol Device:D_Schottky
- added FB30, FB31: 600R@100MHz provisional, symbol Device:L_Ferrite
- added R300: 10k reset pull-up, Resistor_SMD:R_0805_2012Metric, symbol Device:R
- added R301: 20k, Resistor_SMD:R_0805_2012Metric, symbol Device:R
- added R302, R304: 10k, Resistor_SMD:R_0805_2012Metric, symbol Device:R
- added R303: 30k, Resistor_SMD:R_0805_2012Metric, symbol Device:R
- added R305, R307: 100k bias, Resistor_SMD:R_0805_2012Metric, symbol Device:R
- added R306, R308: 1.5k, Resistor_SMD:R_0805_2012Metric, symbol Device:R
- added R340, R341, R347, R348, R354, R355: 7.5k, Resistor_SMD:R_0805_2012Metric, symbol Device:R
- added R342, R343, R349, R350, R356, R357: 360R, Resistor_SMD:R_0805_2012Metric, symbol Device:R
- added R344, R345, R351, R352, R358, R359: 5.6k, Resistor_SMD:R_0805_2012Metric, symbol Device:R
- added R346, R353, R360: 47R output, Resistor_SMD:R_0805_2012Metric, symbol Device:R
- added TP300: CODEC_OVF, symbol Connector:TestPoint
- added TP301: CODEC_ZERO, symbol Connector:TestPoint
- added TP302: CODEC_RST_HW_N, symbol Connector:TestPoint
- added TP303: ADC_ANALOG_IN, symbol Connector:TestPoint
- added TP304: ADC_VIN1_P, symbol Connector:TestPoint
- added TP305: ADC_VIN1_N, symbol Connector:TestPoint
- added TP306: MEMORY_DAC, symbol Connector:TestPoint
- added TP307: GHOST_DAC, symbol Connector:TestPoint
- added TP308: RETURN_DAC, symbol Connector:TestPoint
- added TP309: CODEC_5V_LOCAL, symbol Connector:TestPoint
- added TP310: CODEC_3V3_LOCAL, symbol Connector:TestPoint
- added U30: PCM3168A, symbol MerrinLab_PrototypeA:PCM3168A_PAP_APPLICATION
- added U31: OPA1679 ADC + MEMORY/GHOST, symbol MerrinLab_PrototypeA:OPA1679_PW_APPLICATION
- added U32: OPA1679 RETURN + SPARES, symbol MerrinLab_PrototypeA:OPA1679_PW_APPLICATION
Connections:
- net ADC_ANALOG_IN: now also R301.1, R303.1, TP303.1
- net CODEC_BCLK: now also U30.36 (BCKDA), U30.7 (BCKAD)
- net CODEC_DIN: now also U30.37 (DIN1)
- net CODEC_DOUT: now also U30.8 (DOUT1)
- net CODEC_LRCLK: now also U30.35 (LRCKDA), U30.6 (LRCKAD)
- net CODEC_MCLK: now also U30.41 (SCKI)
- net CODEC_MUTE_N: now also D301.1 (K)
- net CODEC_RESET_N: now also D300.1 (K)
- net CTRL_I2C_SCL: now also U30.42 (MC/SCL/FMT)
- net CTRL_I2C_SDA: now also U30.43 (MDI/SDA/DEMP)
- net GHOST_DAC: now also R353.2, TP307.1
- net MEMORY_DAC: now also R346.2, TP306.1
- net RAIL_3V3: now also FB31.1
- net RAIL_5V_CODEC: now also FB30.1
- net RETURN_DAC: now also R360.2, TP308.1
- new net ADC2_UNUSED: C312.1, U30.53 (VIN2-), U30.54 (VIN2+)
- new net ADC3_UNUSED: C313.1, U30.55 (VIN3-), U30.56 (VIN3+)
- new net ADC4_UNUSED: C314.1, U30.57 (VIN4-), U30.58 (VIN4+)
- new net ADC5_UNUSED: C315.1, U30.61 (VIN5-), U30.62 (VIN5+)
- new net ADC6_UNUSED: C316.1, U30.63 (VIN6-), U30.64 (VIN6+)
- new net ADC_NEG_AC: C332.2, R307.2, R308.1
- new net ADC_NEG_BUF: C332.1, R304.1, U31.7 (OUT_B)
- new net ADC_NEG_SUM: R303.2, R304.2, U31.6 (IN_B-)
- new net ADC_POS_AC: C330.2, R305.2, R306.1
- new net ADC_POS_BUF: C330.1, U31.1 (OUT_A), U31.2 (IN_A-)
- new net ADC_POS_DIV: R301.2, R302.1, U31.3 (IN_A+)
- new net ADC_VIN1_N: C333.1, R308.2, TP305.1, U30.51 (VIN1-)
- new net ADC_VIN1_P: C331.1, R306.2, TP304.1, U30.52 (VIN1+)
- new net CODEC_3V3_LOCAL: C301.1, C306.1, C307.1, FB31.2, R300.1, TP310.1, U30.12 (VDD2), U30.46 (VDD1)
- new net CODEC_5V_LOCAL: C300.1, C302.1, C303.1, C304.1, C305.1, FB30.2, TP309.1, U30.14 (VCCDA1), U30.3 (VCCAD2), U30.34 (VCCDA2), U30.49 (VCCAD1)
- new net CODEC_OVF: TP300.1, U30.5 (OVF)
- new net CODEC_RST_HW_N: D300.2 (A), D301.2 (A), R300.2, TP302.1, U30.4 (RST)
- new net CODEC_VCOMAD: C308.1, C331.2, C333.2, R305.1, R307.1, U30.1 (VCOMAD)
- new net CODEC_VCOMDA: C309.1, U30.15 (VCOMDA)
- new net CODEC_VREFAD1: C310.1, U30.59 (VREFAD1)
- new net CODEC_VREFAD2: C311.1, U30.60 (VREFAD2)
- new net CODEC_ZERO: TP301.1, U30.13 (ZERO)
- new net GHOST_DAC_N: C346.1, U30.30 (VOUT2-)
- new net GHOST_DAC_P: C345.1, U30.29 (VOUT2+)
- new net GHOST_FILT_N: C347.2, R348.2, R350.1
- new net GHOST_FILT_P: C347.1, R347.2, R349.1
- new net GHOST_OP_N: C349.2, R350.2, R352.2, U31.13 (IN_D-)
- new net GHOST_OP_OUT: C349.1, R352.1, R353.1, U31.14 (OUT_D)
- new net GHOST_OP_P: C348.1, R349.2, R351.1, U31.12 (IN_D+)
- new net GHOST_RAW_N: C346.2, R348.1
- new net GHOST_RAW_P: C345.2, R347.1
- new net GND: C300.2, C301.2, C302.2, C303.2, C304.2, C305.2, C306.2, C307.2, C308.2, C309.2, C310.2, C311.2, C312.2, C313.2, C314.2, C315.2, C316.2, C320.2, C321.2, C322.2, C323.2, C324.2, C325.2, C326.2, C327.2, C343.2, C348.2, C353.2, R302.2, R344.2, R351.2, R358.2, U30.11 (DGND2), U30.16 (AGNDDA1), U30.2 (AGNDAD2), U30.33 (AGNDDA2), U30.38 (DIN2), U30.39 (DIN3), U30.40 (DIN4), U30.44 (MDO/ADR1/MD1), U30.45 (MS/ADR0/MD0), U30.47 (DGND1), U30.48 (MODE), U30.50 (AGNDAD1), U30.65 (POWERPAD), U31.5 (IN_B+), U32.10 (IN_C+), U32.12 (IN_D+), U32.5 (IN_B+)
- new net MEMORY_DAC_N: C341.1, U30.32 (VOUT1-)
- new net MEMORY_DAC_P: C340.1, U30.31 (VOUT1+)
- new net MEM_FILT_N: C342.2, R341.2, R343.1
- new net MEM_FILT_P: C342.1, R340.2, R342.1
- new net MEM_OP_N: C344.2, R343.2, R345.2, U31.9 (IN_C-)
- new net MEM_OP_OUT: C344.1, R345.1, R346.1, U31.8 (OUT_C)
- new net MEM_OP_P: C343.1, R342.2, R344.1, U31.10 (IN_C+)
- new net MEM_RAW_N: C341.2, R341.1
- new net MEM_RAW_P: C340.2, R340.1
- new net RAIL_N12: C321.1, C323.1, C325.1, C327.1, U31.11 (V-), U32.11 (V-)
- new net RAIL_P12: C320.1, C322.1, C324.1, C326.1, U31.4 (V+), U32.4 (V+)
- new net RETURN_DAC_N: C351.1, U30.28 (VOUT3-)
- new net RETURN_DAC_P: C350.1, U30.27 (VOUT3+)
- new net RETURN_FILT_N: C352.2, R355.2, R357.1
- new net RETURN_FILT_P: C352.1, R354.2, R356.1
- new net RETURN_OP_N: C354.2, R357.2, R359.2, U32.2 (IN_A-)
- new net RETURN_OP_OUT: C354.1, R359.1, R360.1, U32.1 (OUT_A)
- new net RETURN_OP_P: C353.1, R356.2, R358.1, U32.3 (IN_A+)
- new net RETURN_RAW_N: C351.2, R355.1
- new net RETURN_RAW_P: C350.2, R354.1
- new net U32B_SPARE_FB: U32.6 (IN_B-), U32.7 (OUT_B)
- new net U32C_SPARE_FB: U32.8 (OUT_C), U32.9 (IN_C-)
- new net U32D_SPARE_FB: U32.13 (IN_D-), U32.14 (OUT_D)
- no-connect marks 0 -> 12
Other:
- note added: "ADC gain contract: each phase = ±ADC_ANALOG_IN / 3. 2 Vpp nominal → 1.333 Vpp differential ≈ −12.6 dBFS; 6 Vpp → 4 Vpp differential ≈ −3.0 dBFS."
- note added: "ADC2–6 differential pins are paired and AC-terminated to AGND; DAC4–8 and DOUT2/3 are explicit no-connects. Firmware keeps inactive channels muted/power-save. VCOM/VREF are local decoupling references only."
- note added: "CODEC_MUTE_N is a hard reset/power-down request through the diode AND gate. PCM soft mute remains I²C-controlled; external SSI2164 attenuation remains the primary wet/Return safety clamp."
- note added: "DAC filters follow TI Figure 61 nominal values: R1 7.5k, R2 5.6k, R3 360R, C1 3.3nF, C2 680pF, gain ≈ 0.747, f−3dB ≈ 53kHz."
- note added: "PCM3168A • DIFFERENTIAL ADC INGRESS • MEMORY / GHOST / RETURN DAC FILTERS"
- note removed: "HIERARCHY / INTERFACE CAPTURE ONLY — CIRCUIT CONTENT NOT YET ACCEPTED"
- title: Memory Core Prototype A — CODEC / CONVERSION -> Memory Core Prototype A — Codec / Conversion

Commit message: Capture ERC-validated output mute protection sheet
Parts:
- removed U32: OPA1679 RETURN + SPARES, symbol MerrinLab_PrototypeA:OPA1679_PW_APPLICATION
- added U32: OPA1679, symbol MerrinLab_PrototypeA:OPA1679_PW_MULTI
Connections:
- net RAIL_N12: now also U32.11 (V-)
- net RAIL_P12: now also U32.4 (V+)
- net RETURN_OP_N: now also U32.2 (IN_A-)
- net RETURN_OP_OUT: now also U32.1 (OUT_A)
- net RETURN_OP_P: now also U32.3 (IN_A+)
Changed lines of the file:
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@@
 	)
 	(symbol
-		(lib_id "MerrinLab_PrototypeA:OPA1679_PW_APPLICATION")
+		(lib_id "MerrinLab_PrototypeA:OPA1679_PW_MULTI")
 		(at 326.39 251.46 0)
 		(unit 1)
@@
 		(fields_autoplaced no)
 		(property "Reference" "U32"
-			(at 326.39 265.43 0.0000)
+			(at 326.39 260.35 0.0000)
 			(effects
 				(font
@@
 			)
 		)
-		(property "Value" "OPA1679 RETURN + SPARES"
-			(at 326.39 237.49 0.0000)
+		(property "Value" "OPA1679"
+			(at 326.39 242.57 0.0000)
 			(effects
 				(font
@@
 			)
 		)
-		(pin "1"
+		(pin "3"
 		)
 		(pin "2"
 		)
-		(pin "3"
-		)
-		(pin "4"
+		(pin "1"
 		)
 		(pin "5"
@@
 		(pin "7"
 		)
-		(pin "8"
+		(pin "10"
 		)
 		(pin "9"
 		)
-		(pin "10"
+		(pin "8"
+		)
+		(pin "12"
+		)
+		(pin "13"
+		)
+		(pin "14"
 		)
 		(pin "11"
 		)
+		(pin "4"
+		)
+		(instances
+			(project "MerrinGriefSynthMemoryCoreA"
+				(path "/ea499acf-881c-477d-99db-4f6dec6846fd/df19c340-b121-418f-9b23-7138949f3072"
+					(reference "U32")
+					(unit 1)
+				)
+			)
+		)
+	)
+	(symbol
+		(lib_id "MerrinLab_PrototypeA:OPA1679_PW_MULTI")
+		(at 361.95 251.46 0)
+		(unit 5)
+		(exclude_from_sim no)
+		(in_bom yes)
+		(on_board yes)
+		(dnp no)
+		(fields_autoplaced no)
+		(property "Reference" "U32"
+			(at 361.95 260.35 0.0000)
+			(effects
+				(font
+					(size 1.27 1.27)
+				)
+				(justify left)
+			)
+		)
+		(property "Value" "OPA1679"
+			(at 361.95 242.57 0.0000)
+			(effects
+				(font
+					(size 1.27 1.27)
+				)
+				(justify left)
+			)
+		)
+		(property "Footprint" ""
+			(at 361.95 251.46 0.0000)
+			(effects
+				(font
+					(size 1.27 1.27)
+				)
+				(hide yes)
+			)
+		)
+		(property "hierarchy_path" "/ea499acf-881c-477d-99db-4f6dec6846fd/df19c340-b121-418f-9b23-7138949f3072"
+			(at 364.49 256.5399 0)
+			(effects
+				(font
+					(size 1.27 1.27)
+				)
+				(justify left)
+			)
+		)
+		(pin "3"
+		)
+		(pin "2"
+		)
+		(pin "1"
+		)
+		(pin "5"
+		)
+		(pin "6"
+		)
+		(pin "7"
+		)
+		(pin "10"
+		)
+		(pin "9"
+		)
+		(pin "8"
+		)
 		(pin "12"
 		)
@@
 		(pin "14"
 		)
+		(pin "11"
+		)
+		(pin "4"
+		)
 		(instances
 			(project "MerrinGriefSynthMemoryCoreA"
 				(path "/ea499acf-881c-477d-99db-4f6dec6846fd/df19c340-b121-418f-9b23-7138949f3072"
 					(reference "U32")
-					(unit 1)
+					(unit 5)
 				)
 			)
@@
 	)
 	(label "RAIL_P12"
-		(at 316.23 250.19 0)
+		(at 372.11 247.65 0)
 		(effects
 			(font
@@
 	)
 	(label "RAIL_N12"
-		(at 336.55 250.19 0)
+		(at 351.79 252.73 0)
 		(effects
 			(font
@@
 	)
 	(label "RETURN_OP_N"
-		(at 316.23 245.11 0)
+		(at 316.23 252.73 0)
 		(effects
 			(font
@@
 	)
 	(label "RETURN_OP_OUT"
-		(at 316.23 242.57 0)
+		(at 336.55 250.19 0)
 		(effects
 			(font
@@
 		)
 	)
-	(label "GND"
-		(at 316.23 255.27 0)
-		(effects
-			(font
-				(size 1.27 1.27)
-			)
-			(justify left bottom)
-		)
-	)
-	(label "U32B_SPARE_FB"
-		(at 316.23 257.81 0)
-		(effects
-			(font
-				(size 1.27 1.27)
-			)
-			(justify left bottom)
-		)
-	)
-	(label "U32B_SPARE_FB"
-		(at 316.23 260.35 0)
-		(effects
-			(font
-				(size 1.27 1.27)
-			)
-			(justify left bottom)
-		)
-	)
-	(label "GND"
-		(at 336.55 247.65 0)
-		(effects
-			(font
-				(size 1.27 1.27)
-			)
-			(justify left bottom)
-		)
-	)
-	(label "U32C_SPARE_FB"
-		(at 336.55 245.11 0)
-		(effects
-			(font
-				(size 1.27 1.27)
-			)
-			(justify left bottom)
-		)
-	)
-	(label "U32C_SPARE_FB"
-		(at 336.55 242.57 0)
-		(effects
-			(font
-				(size 1.27 1.27)
-			)
-			(justify left bottom)
-		)
-	)
-	(label "GND"
-		(at 336.55 255.27 0)
-		(effects
-			(font
-				(size 1.27 1.27)
-			)
-			(justify left bottom)
-		)
-	)
-	(label "U32D_SPARE_FB"
-		(at 336.55 257.81 0)
-		(effects
-			(font
-				(size 1.27 1.27)
-			)
-			(justify left bottom)
-		)
-	)
-	(label "U32D_SPARE_FB"
-		(at 336.55 260.35 0)
-		(effects
-			(font
-				(size 1.27 1.27)
-			)
-			(justify left bottom)
-		)
-	)
 	(label "ADC_ANALOG_IN"
 		(at 50.8 173.99 0)
@@
 	)
 	(hierarchical_label "CTRL_I2C_SDA"
-		(shape input)
+		(shape bidirectional)
 		(at 20.32 87.63 0.0000)
 		(effects
@@
 	)
 	(hierarchical_label "CODEC_DOUT"
-		(shape input)
+		(shape output)
 		(at 391.16 30.48 0.0000)
 		(effects
@@
 	)
 	(hierarchical_label "MEMORY_DAC"
-		(shape input)
+		(shape output)
 		(at 391.16 43.18 0.0000)
 		(effects
@@
 	)
 	(hierarchical_label "GHOST_DAC"
-		(shape input)
+		(shape output)
 		(at 391.16 55.88 0.0000)
 		(effects
@@
 	)
 	(hierarchical_label "RETURN_DAC"
-		(shape input)
+		(shape output)
 		(at 391.16 68.58 0.0000)
 		(effects
