File: hardware/memory-core-prototype-a/08_CONTROLS_STATE.kicad_sch (KiCad schematic)
At the start: 1 part, among them J908 SHEET_INTERFACE_NOT_FITTED

Commit message: Capture ERC-validated controls and state sheet
Parts:
- removed J908: SHEET_INTERFACE_NOT_FITTED, symbol Connector_Generic:Conn_01x13
- added C101, C102, C103: 10nF debounce/RF, Capacitor_SMD:C_0805_2012Metric, symbol Device:C
- added C81, C83: 100nF, Capacitor_SMD:C_0805_2012Metric, symbol Device:C
- added C82: 10µF, Capacitor_SMD:C_0805_2012Metric, symbol Device:C
- added C84, C85, C86, C87: 10nF, Capacitor_SMD:C_0805_2012Metric, symbol Device:C
- added C91, C92, C93, C94, C95, C96, C97, C98: 100nF ADC filter, Capacitor_SMD:C_0805_2012Metric, symbol Device:C
- added D21: SLS-1 R, symbol MerrinLab_PrototypeA:LED_AK
- added D22: SLS-1 G, symbol MerrinLab_PrototypeA:LED_AK
- added D23: SLS-1 B, symbol MerrinLab_PrototypeA:LED_AK
- added D24: SLS-1 AUX, symbol MerrinLab_PrototypeA:LED_AK
- added D81: BAT54-class fault clamp, symbol Device:D_Schottky
- added D82, D83, D84, D85, D86, D87, D88, D89: BAT54-class, symbol Device:D_Schottky
- added Q1, Q2, Q3, Q4: NPN LED DRIVER, symbol MerrinLab_PrototypeA:Q_NPN_BCE
- added R101, R102, R103: 100k pull-up, Resistor_SMD:R_0805_2012Metric, symbol Device:R
- added R111, R112, R113: 1k isolate, Resistor_SMD:R_0805_2012Metric, symbol Device:R
- added R121, R122, R123, R124: 10k base, Resistor_SMD:R_0805_2012Metric, symbol Device:R
- added R131, R132, R133, R134: 100k base pull-down, Resistor_SMD:R_0805_2012Metric, symbol Device:R
- added R141, R142, R143, R144: 1k LED limit, Resistor_SMD:R_0805_2012Metric, symbol Device:R
- added R150, R151, R152, R153, R154, R155, R156, R157: 1k ADC isolate, Resistor_SMD:R_0805_2012Metric, symbol Device:R
- added R81, R82: 4.7k, Resistor_SMD:R_0805_2012Metric, symbol Device:R
- added R83: 100k RDY pull-up, Resistor_SMD:R_0805_2012Metric, symbol Device:R
- added R84: 100k default-safe pull-down, Resistor_SMD:R_0805_2012Metric, symbol Device:R
- added R85: 10k release feed, Resistor_SMD:R_0805_2012Metric, symbol Device:R
- added R86, R87, R88, R89: 1k, Resistor_SMD:R_0805_2012Metric, symbol Device:R
- added R90, R91, R92, R93: 1k output isolate, Resistor_SMD:R_0805_2012Metric, symbol Device:R
- added RV1: MEMORY TIME, symbol MerrinLab_PrototypeA:R_POT_123
- added RV2: MEMORY FADE, symbol MerrinLab_PrototypeA:R_POT_123
- added RV3: MEMORY BLUR, symbol MerrinLab_PrototypeA:R_POT_123
- added RV4: GHOST DISTANCE, symbol MerrinLab_PrototypeA:R_POT_123
- added RV5: GHOST DRIFT, symbol MerrinLab_PrototypeA:R_POT_123
- added RV6: GHOST PRESENCE, symbol MerrinLab_PrototypeA:R_POT_123
- added RV7: RETURN AMOUNT, symbol MerrinLab_PrototypeA:R_POT_123
- added RV8: PRESENT / WET, symbol MerrinLab_PrototypeA:R_POT_123
- added SW2: SERVICE TEST, symbol Switch:SW_Push
- added SW3: RESET / CLEAR, symbol Switch:SW_Push
- added SW4: SAFE MUTE, symbol Switch:SW_Push
- added TP81: MCP4728_RDY_N, symbol Connector:TestPoint
- added TP82: SAFE_SELECTOR_SEL, symbol Connector:TestPoint
- added TP83: VCA_MEMORY_CTRL, symbol Connector:TestPoint
- added TP84: VCA_GHOST_CTRL, symbol Connector:TestPoint
- added TP85: VCA_RETURN_CTRL, symbol Connector:TestPoint
- added TP86: VCA_WET_CTRL, symbol Connector:TestPoint
- added TP87: RAIL_3V3, symbol Connector:TestPoint
- added TP88: GND, symbol Connector:TestPoint
- added U6: MCP4728 — VCA CONTROL, symbol MerrinLab_PrototypeA:MCP4728_UN
- added U7: TMUX1574 — SAFE SELECTOR, symbol MerrinLab_PrototypeA:TMUX1574PW
Connections:
- net CTRL_I2C_SCL: now also R81.2, U6.2 (SCL)
- net CTRL_I2C_SDA: now also R82.2, U6.3 (SDA)
- net HARDWARE_FAULT_N: now also D81.1 (K)
- net RAIL_3V3: now also C81.1, C82.1, C83.1, D82.1 (K), D84.1 (K), D86.1 (K), D88.1 (K), R101.1, R102.1, R103.1, R141.2, R142.2, R143.2, R144.2, R81.1, R82.1, R83.1, RV1.3 (END_B), RV2.3 (END_B), RV3.3 (END_B), RV4.3 (END_B), RV5.3 (END_B), RV6.3 (END_B), RV7.3 (END_B), RV8.3 (END_B), TP87.1, U6.1 (VDD), U7.11 (S3A), U7.14 (S4A), U7.16 (VDD), U7.2 (S1A), U7.5 (S2A)
- net SAFE_CONTROL_RELEASE: now also R85.1
- net STATE_LED_AUX: now also R124.1
- net STATE_LED_B: now also R123.1
- net STATE_LED_G: now also R122.1
- net STATE_LED_R: now also R121.1
- net VCA_GHOST_CTRL: now also R91.2, TP84.1
- net VCA_MEMORY_CTRL: now also R90.2, TP83.1
- net VCA_RETURN_CTRL: now also R92.2, TP85.1
- net VCA_WET_CTRL: now also R93.2, TP86.1
- new net DAC_GHOST_CTRL: U6.7 (VOUT_B), U7.6 (S2B)
- new net DAC_MEMORY_CTRL: U6.6 (VOUT_A), U7.3 (S1B)
- new net DAC_RETURN_CTRL: U6.8 (VOUT_C), U7.10 (S3B)
- new net DAC_WET_CTRL: U6.9 (VOUT_D), U7.13 (S4B)
- new net GHOST_CTRL_FILTERED: C85.1, D84.2 (A), D85.1 (K), R87.2, R91.1
- new net GND: C101.2, C102.2, C103.2, C81.2, C82.2, C83.2, C84.2, C85.2, C86.2, C87.2, C91.2, C92.2, C93.2, C94.2, C95.2, C96.2, C97.2, C98.2, D83.2 (A), D85.2 (A), D87.2 (A), D89.2 (A), Q1.3 (E), Q2.3 (E), Q3.3 (E), Q4.3 (E), R131.2, R132.2, R133.2, R134.2, R84.2, RV1.1 (END_A), RV2.1 (END_A), RV3.1 (END_A), RV4.1 (END_A), RV5.1 (END_A), RV6.1 (END_A), RV7.1 (END_A), RV8.1 (END_A), SW2.2, SW3.2, SW4.2, TP88.1, U6.10 (VSS), U6.4 (LDAC), U7.15 (EN_N), U7.8 (GND)
- new net MCP4728_RDY_N: R83.2, TP81.1, U6.5 (RDY_BSY_N)
- new net MEMORY_CTRL_FILTERED: C84.1, D82.2 (A), D83.1 (K), R86.2, R90.1
- new net MUX_GHOST_CTRL: R87.1, U7.7 (D2)
- new net MUX_MEMORY_CTRL: R86.1, U7.4 (D1)
- new net MUX_RETURN_CTRL: R88.1, U7.9 (D3)
- new net MUX_WET_CTRL: R89.1, U7.12 (D4)
- new net PANEL_GHOST_DISTANCE: C94.1, R153.2
- new net PANEL_GHOST_DISTANCE_RAW: R153.1, RV4.2 (WIPER)
- new net PANEL_GHOST_DRIFT: C95.1, R154.2
- new net PANEL_GHOST_DRIFT_RAW: R154.1, RV5.2 (WIPER)
- new net PANEL_GHOST_PRESENCE: C96.1, R155.2
- new net PANEL_GHOST_PRESENCE_RAW: R155.1, RV6.2 (WIPER)
- new net PANEL_MEMORY_BLUR: C93.1, R152.2
- new net PANEL_MEMORY_BLUR_RAW: R152.1, RV3.2 (WIPER)
- new net PANEL_MEMORY_FADE: C92.1, R151.2
- new net PANEL_MEMORY_FADE_RAW: R151.1, RV2.2 (WIPER)
- new net PANEL_MEMORY_TIME: C91.1, R150.2
- new net PANEL_MEMORY_TIME_RAW: R150.1, RV1.2 (WIPER)
- new net PANEL_PRESENT_WET: C98.1, R157.2
- new net PANEL_PRESENT_WET_RAW: R157.1, RV8.2 (WIPER)
- new net PANEL_RETURN_AMOUNT: C97.1, R156.2
- new net PANEL_RETURN_AMOUNT_RAW: R156.1, RV7.2 (WIPER)
- new net RESET_CLEAR: C102.1, R112.2
- new net RESET_CLEAR_RAW_N: R102.2, R112.1, SW3.1
- new net RETURN_CTRL_FILTERED: C86.1, D86.2 (A), D87.1 (K), R88.2, R92.1
- new net SAFE_MUTE: C103.1, R113.2
- new net SAFE_MUTE_RAW_N: R103.2, R113.1, SW4.1
- new net SAFE_SELECTOR_SEL: D81.2 (A), R84.1, R85.2, TP82.1, U7.1 (SEL)
- new net SERVICE_TEST: C101.1, R111.2
- new net SERVICE_TEST_RAW_N: R101.2, R111.1, SW2.1
- new net STATE_AUX_BASE: Q4.1 (B), R124.2, R134.1
- new net STATE_AUX_COLLECTOR: D24.1 (K), Q4.2 (C)
- new net STATE_AUX_LED_ANODE: D24.2 (A), R144.1
- new net STATE_B_BASE: Q3.1 (B), R123.2, R133.1
- new net STATE_B_COLLECTOR: D23.1 (K), Q3.2 (C)
- new net STATE_B_LED_ANODE: D23.2 (A), R143.1
- new net STATE_G_BASE: Q2.1 (B), R122.2, R132.1
- new net STATE_G_COLLECTOR: D22.1 (K), Q2.2 (C)
- new net STATE_G_LED_ANODE: D22.2 (A), R142.1
- new net STATE_R_BASE: Q1.1 (B), R121.2, R131.1
- new net STATE_R_COLLECTOR: D21.1 (K), Q1.2 (C)
- new net STATE_R_LED_ANODE: D21.2 (A), R141.1
- new net WET_CTRL_FILTERED: C87.1, D88.2 (A), D89.1 (K), R89.2, R93.1
Other:
- note added: "MCP4728 LDAC is tied low: accepted writes update at the final-byte acknowledge. EEPROM must request 0xFFF attenuation, but TMUX1574 remains the authoritative safety layer."
- note added: "NORMAL CONTROL CANNOT OVERRIDE HARDWARE FAULT • +3.3 V = SSI2164 ATTENUATION"
- note added: "Panel controls and LEDs are electrically captured only. Final panel mechanics and footprints remain blocked."
- note added: "SEL low = +3.3 V safe attenuation. SEL high = MCP4728 normal control. HARDWARE_FAULT_N low clamps SEL low through D81; MCU release alone cannot override fault."
- note removed: "HIERARCHY / INTERFACE CAPTURE ONLY — CIRCUIT CONTENT NOT YET ACCEPTED"
- title: Memory Core Prototype A — CONTROLS / STATE / SAFE SELECTOR -> Memory Core Prototype A — Controls / State / Safe Selector

Commit message: Complete final integrated schematic review
Changed lines of the file:
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@@
 	)
 	(hierarchical_label "CTRL_I2C_SDA"
-		(shape input)
+		(shape bidirectional)
 		(at 20.32 48.26 0.0000)
 		(effects
@@
 	)
 	(hierarchical_label "VCA_MEMORY_CTRL"
-		(shape input)
+		(shape output)
 		(at 391.16 35.56 0.0000)
 		(effects
@@
 	)
 	(hierarchical_label "VCA_GHOST_CTRL"
-		(shape input)
+		(shape output)
 		(at 391.16 41.91 0.0000)
 		(effects
@@
 	)
 	(hierarchical_label "VCA_RETURN_CTRL"
-		(shape input)
+		(shape output)
 		(at 391.16 48.26 0.0000)
 		(effects
@@
 	)
 	(hierarchical_label "VCA_WET_CTRL"
-		(shape input)
+		(shape output)
 		(at 391.16 54.61 0.0000)
 		(effects
@@
 	)
 	(hierarchical_label "PANEL_MEMORY_TIME"
-		(shape input)
+		(shape output)
 		(at 391.16 60.96 0.0000)
 		(effects
@@
 	)
 	(hierarchical_label "PANEL_MEMORY_FADE"
-		(shape input)
+		(shape output)
 		(at 391.16 67.31 0.0000)
 		(effects
@@
 	)
 	(hierarchical_label "PANEL_MEMORY_BLUR"
-		(shape input)
+		(shape output)
 		(at 391.16 73.66 0.0000)
 		(effects
@@
 	)
 	(hierarchical_label "PANEL_GHOST_DISTANCE"
-		(shape input)
+		(shape output)
 		(at 391.16 80.01 0.0000)
 		(effects
@@
 	)
 	(hierarchical_label "PANEL_GHOST_DRIFT"
-		(shape input)
+		(shape output)
 		(at 391.16 86.36 0.0000)
 		(effects
@@
 	)
 	(hierarchical_label "PANEL_GHOST_PRESENCE"
-		(shape input)
+		(shape output)
 		(at 391.16 92.71 0.0000)
 		(effects
@@
 	)
 	(hierarchical_label "PANEL_RETURN_AMOUNT"
-		(shape input)
+		(shape output)
 		(at 391.16 99.06 0.0000)
 		(effects
@@
 	)
 	(hierarchical_label "PANEL_PRESENT_WET"
-		(shape input)
+		(shape output)
 		(at 391.16 105.41 0.0000)
 		(effects
@@
 	)
 	(hierarchical_label "SERVICE_TEST"
-		(shape input)
+		(shape output)
 		(at 391.16 111.76 0.0000)
 		(effects
@@
 	)
 	(hierarchical_label "RESET_CLEAR"
-		(shape input)
+		(shape output)
 		(at 391.16 118.11 0.0000)
 		(effects
@@
 	)
 	(hierarchical_label "SAFE_MUTE"
-		(shape input)
+		(shape output)
 		(at 391.16 124.46 0.0000)
 		(effects
