File: hardware/memory-core-prototype-a/07_OUTPUT_MUTE_PROTECTION.kicad_sch (KiCad schematic)
At the start: 32 parts, among them J70 WQP518MA / THONKICONN OUTPUT, Q70 J113 OUTPUT MUTE SHUNT, Q71 MMBT3904 fault inverter provi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, U32 OPA1679, U70 LTV-817S-CLASS FAIL-MUTE

Commit message: Apply validated exact output mute parts
Parts:
- C710: value 1uF mute ramp -> 100nF C0G 50V mute timing
- Q70: value J113 OUTPUT MUTE SHUNT -> MMBFJ113 OUTPUT MUTE SHUNT; footprint (none) -> Package_TO_SOT_SMD:SOT-23; symbol MerrinLab_PrototypeA:J113_SHUNT_APPLICATION -> MerrinLab_PrototypeA:MMBFJ113_APPLICATION
- Q71: value MMBT3904 fault inverter provisional -> PMV20XNE HEALTHY-RELEASE DRIVER; footprint (none) -> Package_TO_SOT_SMD:SOT-23; symbol MerrinLab_PrototypeA:NPN_FAULT_INVERTER_APPLICATION -> MerrinLab_PrototypeA:PMV20XNE_APPLICATION
- R703: value 10k mute isolation -> 120k 1% mute isolation
- R711: value 10k fault inverter base -> 10k fault gate series
- R712: value 100k fault base pull-down -> 100k fault gate pull-down
- R713: value 2.2k +12V fault pull-up -> 820R 1% optocoupler LED series A
- R714: value 3.3k optocoupler LED -> 1k 1% optocoupler LED series B
- R715: value 100k controlled release -> 10k 1% negative release
- R716: value 1M power-off mute -> 100k 1% fail-mute pull
- U70: value LTV-817S-CLASS FAIL-MUTE -> VO617A-3X007T HEALTHY RELEASE; footprint (none) -> Package_DIP:SMDIP-4_W7.62mm; symbol MerrinLab_PrototypeA:LTV817S_MUTE_APPLICATION -> MerrinLab_PrototypeA:VO617A_3X007T_APPLICATION
Connections:
- net GND: now also Q70.2 (SOURCE), Q71.2 (SOURCE); no longer Q70.3 (S), Q71.3 (EMITTER), U70.2 (LED_K), U70.4 (COLLECTOR)
- net MUTE_GATE: now also Q70.3 (GATE), U70.4 (COLLECTOR); no longer Q70.2 (G), R715.2, U70.3 (EMITTER)
- net FAULT_INV_BASE renamed FAULT_GATE
- net MUTE_FAULT_HIGH renamed MUTE_LED_SUPPLY
- net MUTE_LED_SUPPLY: no longer Q71.2 (COLLECTOR)
- new net MUTE_LED_K: Q71.3 (DRAIN), U70.2 (LED_K)
- new net RELEASE_SINK: R715.2, U70.3 (EMITTER)
Other:
- note added: "BOUNDARY All mix, level, mute, output-protection and jack nodes remain local to sheet 07. No audio or control net is exported; Q70/Q71/U70 package mappings are accepted, while jack mechanics and PCB work remain blocked."
- note added: "DIRECT + WET HALF-SUM • OUTPUT LEVEL • HEALTHY-RELEASE FAIL-MUTE • PROTECTED MONO OUT"
- note added: "EXACT FAIL-MUTE CONTRACT Healthy HARDWARE_FAULT_N drives PMV20XNE and VO617A-3X007T, connecting the negative release path. Fault or +12 V loss removes release drive; 100k/100nF returns MUTE_GATE toward 0 V and crosses -3 V in about 12.6 ms. 120k isolation with 100 ohm worst JFET on-resistance calculates better than 60 dB static attenuation; bench proof remains Gate C."
- note removed: "BOUNDARY All mix, level, mute, output-protection and jack nodes remain local to sheet 07. No audio or control net is exported from this sheet; physical jack/footprint acceptance remains blocked."
- note removed: "DIRECT + WET HALF-SUM • OUTPUT LEVEL • FAIL-MUTED JFET • PROTECTED MONO OUT"
- note removed: "FAIL-MUTE CONTRACT Fault/undefined HARDWARE_FAULT_N lights U70 and clamps MUTE_GATE toward 0 V. Healthy release approaches -10.91 V from RAIL_N12 with about 90.9 ms RC time constant. At 50% assumed CTR, the first-pass fault-clamp estimate is 12.7 ms; exact optocoupler/JFET parts remain a later measured gate."
Changed lines of the file:
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@@
 		(company "MerrinLab")
 		(comment 1 "U32 units B/C/D complete the physical OPA1679 whose A/power units remain on sheet 03.")
-		(comment 2 "Output jack and active-device footprints remain blocked pending independent review.")
+		(comment 2 "Q70/Q71/U70 exact parts and package footprints verified; PCB placement remains blocked.")
 	)
 	(symbol
@@
 			)
 		)
-		(property "Value" "10k mute isolation"
+		(property "Value" "120k 1% mute isolation"
 			(at 233.68 124.46 90)
 			(effects
@@
 	)
 	(symbol
-		(lib_id "MerrinLab_PrototypeA:J113_SHUNT_APPLICATION")
+		(lib_id "MerrinLab_PrototypeA:MMBFJ113_APPLICATION")
 		(at 264.16 147.32 0)
 		(unit 1)
@@
 			)
 		)
-		(property "Value" "J113 OUTPUT MUTE SHUNT"
+		(property "Value" "MMBFJ113 OUTPUT MUTE SHUNT"
 			(at 264.16 137.16 0.0000)
 			(effects
@@
 			)
 		)
-		(property "Footprint" ""
+		(property "Footprint" "Package_TO_SOT_SMD:SOT-23"
 			(at 264.16 147.32 0.0000)
 			(effects
@@
 			)
 		)
-		(property "Value" "10k fault inverter base"
+		(property "Value" "10k fault gate series"
 			(at 91.44 198.12 90)
 			(effects
@@
 			)
 		)
-		(property "Value" "100k fault base pull-down"
+		(property "Value" "100k fault gate pull-down"
 			(at 106.68 213.36 90)
 			(effects
@@
 	)
 	(symbol
-		(lib_id "MerrinLab_PrototypeA:NPN_FAULT_INVERTER_APPLICATION")
+		(lib_id "MerrinLab_PrototypeA:PMV20XNE_APPLICATION")
 		(at 132.08 198.12 0)
 		(unit 1)
@@
 			)
 		)
-		(property "Value" "MMBT3904 fault inverter provisional"
+		(property "Value" "PMV20XNE HEALTHY-RELEASE DRIVER"
 			(at 132.08 187.96 0.0000)
 			(effects
@@
 			)
 		)
-		(property "Footprint" ""
+		(property "Footprint" "Package_TO_SOT_SMD:SOT-23"
 			(at 132.08 198.12 0.0000)
 			(effects
@@
 			)
 		)
-		(property "Value" "2.2k +12V fault pull-up"
+		(property "Value" "820R 1% optocoupler LED series A"
 			(at 154.94 182.88 90)
 			(effects
@@
 			)
 		)
-		(property "Value" "3.3k optocoupler LED"
+		(property "Value" "1k 1% optocoupler LED series B"
 			(at 170.18 198.12 90)
 			(effects
@@
 	)
 	(symbol
-		(lib_id "MerrinLab_PrototypeA:LTV817S_MUTE_APPLICATION")
+		(lib_id "MerrinLab_PrototypeA:VO617A_3X007T_APPLICATION")
 		(at 203.2 198.12 0)
 		(unit 1)
@@
 			)
 		)
-		(property "Value" "LTV-817S-CLASS FAIL-MUTE"
+		(property "Value" "VO617A-3X007T HEALTHY RELEASE"
 			(at 203.2 187.96 0.0000)
 			(effects
@@
 			)
 		)
-		(property "Footprint" ""
+		(property "Footprint" "Package_DIP:SMDIP-4_W7.62mm"
 			(at 203.2 198.12 0.0000)
 			(effects
@@
 			)
 		)
-		(property "Value" "100k controlled release"
+		(property "Value" "10k 1% negative release"
 			(at 238.76 182.88 90)
 			(effects
@@
 			)
 		)
-		(property "Value" "1M power-off mute"
+		(property "Value" "100k 1% fail-mute pull"
 			(at 254 198.12 90)
 			(effects
@@
 			)
 		)
-		(property "Value" "1uF mute ramp"
+		(property "Value" "100nF C0G 50V mute timing"
 			(at 269.875 195.58 0.0000)
 			(effects
@@
 		)
 	)
-	(label "FAULT_INV_BASE"
+	(label "FAULT_GATE"
 		(at 91.44 201.93 0)
 		(effects
@@
 		)
 	)
-	(label "FAULT_INV_BASE"
+	(label "FAULT_GATE"
 		(at 106.68 209.55 0)
 		(effects
@@
 		)
 	)
-	(label "FAULT_INV_BASE"
+	(label "FAULT_GATE"
 		(at 121.92 195.58 0)
 		(effects
@@
 		)
 	)
-	(label "MUTE_FAULT_HIGH"
+	(label "MUTE_LED_K"
 		(at 142.24 193.04 0)
 		(effects
@@
 		)
 	)
-	(label "MUTE_FAULT_HIGH"
+	(label "MUTE_LED_SUPPLY"
 		(at 154.94 186.69 0)
 		(effects
@@
 		)
 	)
-	(label "MUTE_FAULT_HIGH"
+	(label "MUTE_LED_SUPPLY"
 		(at 170.18 194.31 0)
 		(effects
@@
 		)
 	)
-	(label "GND"
+	(label "MUTE_LED_K"
 		(at 193.04 198.12 0)
 		(effects
@@
 		)
 	)
+	(label "RELEASE_SINK"
+		(at 213.36 198.12 0)
+		(effects
+			(font
+				(size 1.27 1.27)
+			)
+			(justify left bottom)
+		)
+	)
 	(label "MUTE_GATE"
-		(at 213.36 198.12 0)
-		(effects
-			(font
-				(size 1.27 1.27)
-			)
-			(justify left bottom)
-		)
-	)
-	(label "GND"
 		(at 213.36 193.04 0)
 		(effects
@@
 		)
 	)
-	(label "MUTE_GATE"
+	(label "RELEASE_SINK"
 		(at 238.76 186.69 0)
 		(effects
@@
 		)
 	)
-	(text "DIRECT + WET HALF-SUM • OUTPUT LEVEL • FAIL-MUTED JFET • PROTECTED MONO OUT"
+	(text "DIRECT + WET HALF-SUM • OUTPUT LEVEL • HEALTHY-RELEASE FAIL-MUTE • PROTECTED MONO OUT"
 		(exclude_from_sim no)
 		(at 20.32 17.78 0.0000)
@@
 		)
 	)
-	(text "FAIL-MUTE CONTRACT\nFault/undefined HARDWARE_FAULT_N lights U70 and clamps MUTE_GATE toward 0 V.\nHealthy release approaches -10.91 V from RAIL_N12 with about 90.9 ms RC time constant.\nAt 50% assumed CTR, the first-pass fault-clamp estimate is 12.7 ms; exact optocoupler/JFET parts remain a later measured gate."
+	(text "EXACT FAIL-MUTE CONTRACT\nHealthy HARDWARE_FAULT_N drives PMV20XNE and VO617A-3X007T, connecting the negative release path.\nFault or +12 V loss removes release drive; 100k/100nF returns MUTE_GATE toward 0 V and crosses -3 V in about 12.6 ms.\n120k isolation with 100 ohm worst JFET on-resistance calculates better than 60 dB static attenuation; bench proof remains Gate C."
 		(exclude_from_sim no)
 		(at 294.64 223.52 0.0000)
@@
 		)
 	)
-	(text "BOUNDARY\nAll mix, level, mute, output-protection and jack nodes remain local to sheet 07.\nNo audio or control net is exported from this sheet; physical jack/footprint acceptance remains blocked."
+	(text "BOUNDARY\nAll mix, level, mute, output-protection and jack nodes remain local to sheet 07.\nNo audio or control net is exported; Q70/Q71/U70 package mappings are accepted, while jack mechanics and PCB work remain blocked."
 		(exclude_from_sim no)
 		(at 218.44 269.24 0.0000)
