File: hardware/memory-core-prototype-a/07_OUTPUT_MUTE_PROTECTION.kicad_sch (KiCad schematic)
At the start: 1 part, among them J907 SHEET_INTERFACE_NOT_FITTED

Commit message: Capture ERC-validated output mute protection sheet
Parts:
- removed J907: SHEET_INTERFACE_NOT_FITTED, symbol Connector_Generic:Conn_01x05
- added C700: 220pF mix bandwidth, Capacitor_SMD:C_0805_2012Metric, symbol Device:C
- added C710: 1uF mute ramp, Capacitor_SMD:C_0805_2012Metric, symbol Device:C
- added C720: 10uF bipolar output AC, symbol Device:C
- added C721: 220pF output RF, Capacitor_SMD:C_0805_2012Metric, symbol Device:C
- added C730: 100nF + rail, Capacitor_SMD:C_0805_2012Metric, symbol Device:C
- added C731: 100nF - rail, Capacitor_SMD:C_0805_2012Metric, symbol Device:C
- added C732: 4.7uF + rail, Capacitor_SMD:C_0805_2012Metric, symbol Device:C
- added C733: 4.7uF - rail, Capacitor_SMD:C_0805_2012Metric, symbol Device:C
- added D701: BAT54-class +rail clamp, symbol Device:D_Schottky
- added D702: BAT54-class -rail clamp, symbol Device:D_Schottky
- added J70: WQP518MA / THONKICONN OUTPUT, symbol MerrinLab_PrototypeA:WQP518MA_APPLICATION
- added Q70: J113 OUTPUT MUTE SHUNT, symbol MerrinLab_PrototypeA:J113_SHUNT_APPLICATION
- added Q71: MMBT3904 fault inverter provisional, symbol MerrinLab_PrototypeA:NPN_FAULT_INVERTER_APPLICATION
- added R700: 40.2k 1% Direct sum, Resistor_SMD:R_0805_2012Metric, symbol Device:R
- added R701: 40.2k 1% Wet sum, Resistor_SMD:R_0805_2012Metric, symbol Device:R
- added R702: 20k 1% half-sum feedback, Resistor_SMD:R_0805_2012Metric, symbol Device:R
- added R703: 10k mute isolation, Resistor_SMD:R_0805_2012Metric, symbol Device:R
- added R711: 10k fault inverter base, Resistor_SMD:R_0805_2012Metric, symbol Device:R
- added R712: 100k fault base pull-down, Resistor_SMD:R_0805_2012Metric, symbol Device:R
- added R713: 2.2k +12V fault pull-up, Resistor_SMD:R_0805_2012Metric, symbol Device:R
- added R714: 3.3k optocoupler LED, Resistor_SMD:R_0805_2012Metric, symbol Device:R
- added R715: 100k controlled release, Resistor_SMD:R_0805_2012Metric, symbol Device:R
- added R716: 1M power-off mute, Resistor_SMD:R_0805_2012Metric, symbol Device:R
- added R720: 1k output protection, Resistor_SMD:R_0805_2012Metric, symbol Device:R
- added R721: 100k output reference, Resistor_SMD:R_0805_2012Metric, symbol Device:R
- added RV700: 10k A OUTPUT LEVEL, symbol MerrinLab_PrototypeA:OUTPUT_LEVEL_POT_APPLICATION
- added TP700: FINAL_MIX, symbol Connector:TestPoint
- added TP701: OUT_PREMUTE, symbol Connector:TestPoint
- added TP702: OUTPUT_TIP, symbol Connector:TestPoint
- added TP703: MUTE_GATE, symbol Connector:TestPoint
- added U32: OPA1679, symbol MerrinLab_PrototypeA:OPA1679_PW_MULTI
- added U70: LTV-817S-CLASS FAIL-MUTE, symbol MerrinLab_PrototypeA:LTV817S_MUTE_APPLICATION
Connections:
- net DIRECT_PRESENT: now also R700.1
- net HARDWARE_FAULT_N: now also R711.1
- net RAIL_N12: now also C731.1, C733.1, D702.1 (K), R715.1
- net RAIL_P12: now also C730.1, C732.1, D701.2 (A), R713.1
- net WET_MIX: now also R701.1
- new net FAULT_INV_BASE: Q71.1 (BASE), R711.2, R712.1
- new net FINAL_MIX: C700.1, R702.1, RV700.3 (HIGH), TP700.1, U32.7 (OUT_B)
- new net FINAL_SUM_NODE: C700.2, R700.2, R701.2, R702.2, U32.6 (IN_B-)
- new net GND: C710.2, C721.2, C730.2, C731.2, C732.2, C733.2, J70.3 (SLEEVE), Q70.3 (S), Q71.3 (EMITTER), R712.2, R716.2, R721.2, RV700.1 (LOW), U32.5 (IN_B+), U70.2 (LED_K), U70.4 (COLLECTOR)
- new net MUTE_FAULT_HIGH: Q71.2 (COLLECTOR), R713.2, R714.1
- new net MUTE_GATE: C710.1, Q70.2 (G), R715.2, R716.1, TP703.1, U70.3 (EMITTER)
- new net MUTE_LED_A: R714.2, U70.1 (LED_A)
- new net MUTE_NODE: Q70.1 (D), R703.2, U32.12 (IN_D+)
- new net OUTPUT_AC: C720.2, R720.1
- new net OUTPUT_LEVEL: RV700.2 (WIPER), U32.10 (IN_C+)
- new net OUTPUT_TIP: C721.1, D701.1 (K), D702.2 (A), J70.1 (TIP), R720.2, R721.1, TP702.1
- new net OUT_PREMUTE: R703.1, TP701.1, U32.8 (OUT_C), U32.9 (IN_C-)
- new net POST_MUTE: C720.1, U32.13 (IN_D-), U32.14 (OUT_D)
- no-connect marks 0 -> 1
Other:
- note added: "BOUNDARY All mix, level, mute, output-protection and jack nodes remain local to sheet 07. No audio or control net is exported from this sheet; physical jack/footprint acceptance remains blocked."
- note added: "DIRECT + WET HALF-SUM • OUTPUT LEVEL • FAIL-MUTED JFET • PROTECTED MONO OUT"
- note added: "FAIL-MUTE CONTRACT Fault/undefined HARDWARE_FAULT_N lights U70 and clamps MUTE_GATE toward 0 V. Healthy release approaches -10.91 V from RAIL_N12 with about 90.9 ms RC time constant. At 50% assumed CTR, the first-pass fault-clamp estimate is 12.7 ms; exact optocoupler/JFET parts remain a later measured gate."
- note added: "OUTPUT GAIN CONTRACT R700 = R701 = 40.2k; R702 = 20.0k. Each branch = 0.4975; two 6.0 Vpp inputs calculate to 5.97 Vpp. The 10k output control only attenuates; normal output remains below 10 Vpp."
- note added: "SHARED OPA1679 CONTRACT U32 unit 1 + power unit 5 remain on sheet 03. U32 units 2/3/4 implement final half-sum, level buffer and post-mute driver here. Exactly seven physical OPA1679 packages remain in Prototype A."
- note added: "U32B FINAL HALF-SUM: pins 5 +, 6 -, 7 OUT"
- note added: "U32C OUTPUT LEVEL BUFFER: pins 10 +, 9 -, 8 OUT"
- note added: "U32D POST-MUTE DRIVER: pins 12 +, 13 -, 14 OUT"
- note removed: "HIERARCHY / INTERFACE CAPTURE ONLY — CIRCUIT CONTENT NOT YET ACCEPTED"
- title: Memory Core Prototype A — OUTPUT / MUTE / PROTECTION -> Memory Core Prototype A — Output / Mute / Protection

Commit message: V5.3: verify sheet 07 output mute exact parts
Verify the Q70 MMBFJ113, Q71 PMV20XNE and U70 VO617A-3X007T physical pin maps, package mappings and powered healthy-release fail-mute topology.

Pin the accepted project-local KiCad footprint geometry to an immutable upstream revision, independently validate all three package mappings, and qualify the calculated electrical claims to their datasheet conditions.

Measured and full-temperature behaviour remains Gate C. PCB placement, routing, fabrication and purchasing remain blocked.
Parts:
- C710: value 1uF mute ramp -> 100nF C0G 50V mute timing
- Q70: value J113 OUTPUT MUTE SHUNT -> MMBFJ113 OUTPUT MUTE SHUNT; footprint (none) -> Package_TO_SOT_SMD:SOT-23; symbol MerrinLab_PrototypeA:J113_SHUNT_APPLICATION -> MerrinLab_PrototypeA:MMBFJ113_APPLICATION
- Q71: value MMBT3904 fault inverter provisional -> PMV20XNE HEALTHY-RELEASE DRIVER; footprint (none) -> Package_TO_SOT_SMD:SOT-23; symbol MerrinLab_PrototypeA:NPN_FAULT_INVERTER_APPLICATION -> MerrinLab_PrototypeA:PMV20XNE_APPLICATION
- R703: value 10k mute isolation -> 120k 1% mute isolation
- R711: value 10k fault inverter base -> 10k fault gate series
- R712: value 100k fault base pull-down -> 100k fault gate pull-down
- R713: value 2.2k +12V fault pull-up -> 820R 1% optocoupler LED series A
- R714: value 3.3k optocoupler LED -> 1k 1% optocoupler LED series B
- R715: value 100k controlled release -> 10k 1% negative release
- R716: value 1M power-off mute -> 100k 1% fail-mute pull
- U70: value LTV-817S-CLASS FAIL-MUTE -> VO617A-3X007T HEALTHY RELEASE; footprint (none) -> Package_DIP:SMDIP-4_W7.62mm; symbol MerrinLab_PrototypeA:LTV817S_MUTE_APPLICATION -> MerrinLab_PrototypeA:VO617A_3X007T_APPLICATION
Connections:
- net GND: now also Q70.2 (SOURCE), Q71.2 (SOURCE); no longer Q70.3 (S), Q71.3 (EMITTER), U70.2 (LED_K), U70.4 (COLLECTOR)
- net MUTE_GATE: now also Q70.3 (GATE), U70.4 (COLLECTOR); no longer Q70.2 (G), R715.2, U70.3 (EMITTER)
- net FAULT_INV_BASE renamed FAULT_GATE
- net MUTE_FAULT_HIGH renamed MUTE_LED_SUPPLY
- net MUTE_LED_SUPPLY: no longer Q71.2 (COLLECTOR)
- new net MUTE_LED_K: Q71.3 (DRAIN), U70.2 (LED_K)
- new net RELEASE_SINK: R715.2, U70.3 (EMITTER)
Other:
- note added: "BOUNDARY All mix, level, mute, output-protection and jack nodes remain local to sheet 07. No audio or control net is exported; Q70/Q71/U70 package mappings are accepted, while jack mechanics and PCB work remain blocked."
- note added: "DIRECT + WET HALF-SUM • OUTPUT LEVEL • HEALTHY-RELEASE FAIL-MUTE • PROTECTED MONO OUT"
- note added: "EXACT FAIL-MUTE CONTRACT Healthy HARDWARE_FAULT_N drives PMV20XNE and VO617A-3X007T, connecting the negative release path. Fault or +12 V loss removes release drive; 100k/100nF returns MUTE_GATE toward 0 V and crosses -3 V in about 12.6 ms. 120k isolation with the 100 ohm MMBFJ113 maximum at TJ = 25 C calculates 61.5 dB static attenuation; temperature, spread and measured mute depth remain Gate C."
- note removed: "BOUNDARY All mix, level, mute, output-protection and jack nodes remain local to sheet 07. No audio or control net is exported from this sheet; physical jack/footprint acceptance remains blocked."
- note removed: "DIRECT + WET HALF-SUM • OUTPUT LEVEL • FAIL-MUTED JFET • PROTECTED MONO OUT"
- note removed: "FAIL-MUTE CONTRACT Fault/undefined HARDWARE_FAULT_N lights U70 and clamps MUTE_GATE toward 0 V. Healthy release approaches -10.91 V from RAIL_N12 with about 90.9 ms RC time constant. At 50% assumed CTR, the first-pass fault-clamp estimate is 12.7 ms; exact optocoupler/JFET parts remain a later measured gate."
Changed lines of the file:
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@@
 		(company "MerrinLab")
 		(comment 1 "U32 units B/C/D complete the physical OPA1679 whose A/power units remain on sheet 03.")
-		(comment 2 "Output jack and active-device footprints remain blocked pending independent review.")
+		(comment 2 "Q70/Q71/U70 exact parts and package footprints verified; PCB placement remains blocked.")
 	)
 	(symbol
@@
 			)
 		)
-		(property "Value" "10k mute isolation"
+		(property "Value" "120k 1% mute isolation"
 			(at 233.68 124.46 90)
 			(effects
@@
 	)
 	(symbol
-		(lib_id "MerrinLab_PrototypeA:J113_SHUNT_APPLICATION")
+		(lib_id "MerrinLab_PrototypeA:MMBFJ113_APPLICATION")
 		(at 264.16 147.32 0)
 		(unit 1)
@@
 			)
 		)
-		(property "Value" "J113 OUTPUT MUTE SHUNT"
+		(property "Value" "MMBFJ113 OUTPUT MUTE SHUNT"
 			(at 264.16 137.16 0.0000)
 			(effects
@@
 			)
 		)
-		(property "Footprint" ""
+		(property "Footprint" "Package_TO_SOT_SMD:SOT-23"
 			(at 264.16 147.32 0.0000)
 			(effects
@@
 			)
 		)
-		(property "Value" "10k fault inverter base"
+		(property "Value" "10k fault gate series"
 			(at 91.44 198.12 90)
 			(effects
@@
 			)
 		)
-		(property "Value" "100k fault base pull-down"
+		(property "Value" "100k fault gate pull-down"
 			(at 106.68 213.36 90)
 			(effects
@@
 	)
 	(symbol
-		(lib_id "MerrinLab_PrototypeA:NPN_FAULT_INVERTER_APPLICATION")
+		(lib_id "MerrinLab_PrototypeA:PMV20XNE_APPLICATION")
 		(at 132.08 198.12 0)
 		(unit 1)
@@
 			)
 		)
-		(property "Value" "MMBT3904 fault inverter provisional"
+		(property "Value" "PMV20XNE HEALTHY-RELEASE DRIVER"
 			(at 132.08 187.96 0.0000)
 			(effects
@@
 			)
 		)
-		(property "Footprint" ""
+		(property "Footprint" "Package_TO_SOT_SMD:SOT-23"
 			(at 132.08 198.12 0.0000)
 			(effects
@@
 			)
 		)
-		(property "Value" "2.2k +12V fault pull-up"
+		(property "Value" "820R 1% optocoupler LED series A"
 			(at 154.94 182.88 90)
 			(effects
@@
 			)
 		)
-		(property "Value" "3.3k optocoupler LED"
+		(property "Value" "1k 1% optocoupler LED series B"
 			(at 170.18 198.12 90)
 			(effects
@@
 	)
 	(symbol
-		(lib_id "MerrinLab_PrototypeA:LTV817S_MUTE_APPLICATION")
+		(lib_id "MerrinLab_PrototypeA:VO617A_3X007T_APPLICATION")
 		(at 203.2 198.12 0)
 		(unit 1)
@@
 			)
 		)
-		(property "Value" "LTV-817S-CLASS FAIL-MUTE"
+		(property "Value" "VO617A-3X007T HEALTHY RELEASE"
 			(at 203.2 187.96 0.0000)
 			(effects
@@
 			)
 		)
-		(property "Footprint" ""
+		(property "Footprint" "Package_DIP:SMDIP-4_W7.62mm"
 			(at 203.2 198.12 0.0000)
 			(effects
@@
 			)
 		)
-		(property "Value" "100k controlled release"
+		(property "Value" "10k 1% negative release"
 			(at 238.76 182.88 90)
 			(effects
@@
 			)
 		)
-		(property "Value" "1M power-off mute"
+		(property "Value" "100k 1% fail-mute pull"
 			(at 254 198.12 90)
 			(effects
@@
 			)
 		)
-		(property "Value" "1uF mute ramp"
+		(property "Value" "100nF C0G 50V mute timing"
 			(at 269.875 195.58 0.0000)
 			(effects
@@
 		)
 	)
-	(label "FAULT_INV_BASE"
+	(label "FAULT_GATE"
 		(at 91.44 201.93 0)
 		(effects
@@
 		)
 	)
-	(label "FAULT_INV_BASE"
+	(label "FAULT_GATE"
 		(at 106.68 209.55 0)
 		(effects
@@
 		)
 	)
-	(label "FAULT_INV_BASE"
+	(label "FAULT_GATE"
 		(at 121.92 195.58 0)
 		(effects
@@
 		)
 	)
-	(label "MUTE_FAULT_HIGH"
+	(label "MUTE_LED_K"
 		(at 142.24 193.04 0)
 		(effects
@@
 		)
 	)
-	(label "MUTE_FAULT_HIGH"
+	(label "MUTE_LED_SUPPLY"
 		(at 154.94 186.69 0)
 		(effects
@@
 		)
 	)
-	(label "MUTE_FAULT_HIGH"
+	(label "MUTE_LED_SUPPLY"
 		(at 170.18 194.31 0)
 		(effects
@@
 		)
 	)
-	(label "GND"
+	(label "MUTE_LED_K"
 		(at 193.04 198.12 0)
 		(effects
@@
 		)
 	)
+	(label "RELEASE_SINK"
+		(at 213.36 198.12 0)
+		(effects
+			(font
+				(size 1.27 1.27)
+			)
+			(justify left bottom)
+		)
+	)
 	(label "MUTE_GATE"
-		(at 213.36 198.12 0)
-		(effects
-			(font
-				(size 1.27 1.27)
-			)
-			(justify left bottom)
-		)
-	)
-	(label "GND"
 		(at 213.36 193.04 0)
 		(effects
@@
 		)
 	)
-	(label "MUTE_GATE"
+	(label "RELEASE_SINK"
 		(at 238.76 186.69 0)
 		(effects
@@
 		)
 	)
-	(text "DIRECT + WET HALF-SUM • OUTPUT LEVEL • FAIL-MUTED JFET • PROTECTED MONO OUT"
+	(text "DIRECT + WET HALF-SUM • OUTPUT LEVEL • HEALTHY-RELEASE FAIL-MUTE • PROTECTED MONO OUT"
 		(exclude_from_sim no)
 		(at 20.32 17.78 0.0000)
@@
 		)
 	)
-	(text "FAIL-MUTE CONTRACT\nFault/undefined HARDWARE_FAULT_N lights U70 and clamps MUTE_GATE toward 0 V.\nHealthy release approaches -10.91 V from RAIL_N12 with about 90.9 ms RC time constant.\nAt 50% assumed CTR, the first-pass fault-clamp estimate is 12.7 ms; exact optocoupler/JFET parts remain a later measured gate."
+	(text "EXACT FAIL-MUTE CONTRACT\nHealthy HARDWARE_FAULT_N drives PMV20XNE and VO617A-3X007T, connecting the negative release path.\nFault or +12 V loss removes release drive; 100k/100nF returns MUTE_GATE toward 0 V and crosses -3 V in about 12.6 ms.\n120k isolation with the 100 ohm MMBFJ113 maximum at TJ = 25 C calculates 61.5 dB static attenuation; temperature, spread and measured mute depth remain Gate C."
 		(exclude_from_sim no)
 		(at 294.64 223.52 0.0000)
@@
 		)
 	)
-	(text "BOUNDARY\nAll mix, level, mute, output-protection and jack nodes remain local to sheet 07.\nNo audio or control net is exported from this sheet; physical jack/footprint acceptance remains blocked."
+	(text "BOUNDARY\nAll mix, level, mute, output-protection and jack nodes remain local to sheet 07.\nNo audio or control net is exported; Q70/Q71/U70 package mappings are accepted, while jack mechanics and PCB work remain blocked."
 		(exclude_from_sim no)
 		(at 218.44 269.24 0.0000)

Commit message: V5.4 — Verify input and output jack exact parts (#47)
Accept the WQP518MA/PJ398SM contact and PCB-footprint geometry, add the numeric project-local jack footprint, assign it to J40 and J70, preserve the blank project-symbol default, record the corrected 1.60 mm nut-only fit, and retain all PCB, panel and purchasing blocks.
Parts:
- J70: footprint (none) -> MerrinLab_PrototypeA:Jack_3.5mm_Thonkiconn_WQP518MA_Numeric
Changed lines of the file:
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@@
 			)
 		)
-		(property "Footprint" ""
+		(property "Footprint" "MerrinLab_PrototypeA:Jack_3.5mm_Thonkiconn_WQP518MA_Numeric"
 			(at 386.08 124.46 0.0000)
 			(effects
