File: hardware/memory-core-prototype-a/04_INPUT_PRESSURE_ABSENCE.kicad_sch (KiCad schematic)
At the start: 1 part, among them J904 SHEET_INTERFACE_NOT_FITTED

Commit message: Capture ERC-validated input Pressure Absence sheet
Parts:
- removed J904: SHEET_INTERFACE_NOT_FITTED, symbol Connector_Generic:Conn_01x07
- added C400: 220pF RF, Capacitor_SMD:C_0805_2012Metric, symbol Device:C
- added C401: 1uF AC coupling, symbol Device:C
- added C402, C406: 100nF + rail, Capacitor_SMD:C_0805_2012Metric, symbol Device:C
- added C403, C407: 100nF - rail, Capacitor_SMD:C_0805_2012Metric, symbol Device:C
- added C404, C408: 4.7uF + rail, Capacitor_SMD:C_0805_2012Metric, symbol Device:C
- added C405, C409: 4.7uF - rail, Capacitor_SMD:C_0805_2012Metric, symbol Device:C
- added C410: 1nF Pressure blur, Capacitor_SMD:C_0805_2012Metric, symbol Device:C
- added D400: BAT54-class +rail clamp, symbol Device:D_Schottky
- added D401: BAT54-class -rail clamp, symbol Device:D_Schottky
- added D402, D403: BAV199-class Pressure clip, symbol Device:D
- added D404: 9.1V gate clamp provisional, symbol Device:D_Zener
- added J40: WQP518MA / THONKICONN INPUT, symbol MerrinLab_PrototypeA:WQP518MA_APPLICATION
- added Q40: J113 ABSENCE SHUNT, symbol MerrinLab_PrototypeA:J113_SHUNT_APPLICATION
- added R400: 1k input protection, Resistor_SMD:R_0805_2012Metric, symbol Device:R
- added R401: 1M input reference, Resistor_SMD:R_0805_2012Metric, symbol Device:R
- added R402: 1M post-coupling bias, Resistor_SMD:R_0805_2012Metric, symbol Device:R
- added R403: 47R direct isolation, Resistor_SMD:R_0805_2012Metric, symbol Device:R
- added R404: 22k Pressure input, Resistor_SMD:R_0805_2012Metric, symbol Device:R
- added R405: 22k Pressure feedback, Resistor_SMD:R_0805_2012Metric, symbol Device:R
- added R406: 30.1k Absence input, Resistor_SMD:R_0805_2012Metric, symbol Device:R
- added R407: 121k -12V offset, Resistor_SMD:R_0805_2012Metric, symbol Device:R
- added R408: 80.6k control gain, Resistor_SMD:R_0805_2012Metric, symbol Device:R
- added R409: 22k gate inverter input, Resistor_SMD:R_0805_2012Metric, symbol Device:R
- added R410: 22k gate inverter feedback, Resistor_SMD:R_0805_2012Metric, symbol Device:R
- added R411: 100k JFET gate stop, Resistor_SMD:R_0805_2012Metric, symbol Device:R
- added R412: 20k shaped input, Resistor_SMD:R_0805_2012Metric, symbol Device:R
- added R413: 20k fixed Return input, Resistor_SMD:R_0805_2012Metric, symbol Device:R
- added R414: 20k Memory feedback, Resistor_SMD:R_0805_2012Metric, symbol Device:R
- added R415: 47R ADC isolation, Resistor_SMD:R_0805_2012Metric, symbol Device:R
- added TP400: INPUT_TIP, symbol Connector:TestPoint
- added TP401: INPUT_PROTECTED, symbol Connector:TestPoint
- added TP402: INPUT_BUFFER, symbol Connector:TestPoint
- added TP403: DIRECT_PRESENT, symbol Connector:TestPoint
- added TP404: PRESSURE_OUT, symbol Connector:TestPoint
- added TP405: ABS_GATE, symbol Connector:TestPoint
- added TP406: SHAPED_PRESENT, symbol Connector:TestPoint
- added TP407: RETURN_FEED, symbol Connector:TestPoint
- added TP408: ADC_ANALOG_IN, symbol Connector:TestPoint
- added U40: OPA1679 INPUT/PRESSURE/SUM, symbol MerrinLab_PrototypeA:OPA1679_PW_APPLICATION
- added U41: OPA1679 ABSENCE/OUTPUT, symbol MerrinLab_PrototypeA:OPA1679_PW_APPLICATION
Connections:
- net ABSENCE_INFLUENCE: now also R406.1
- net ADC_ANALOG_IN: now also R415.2, TP408.1
- net DIRECT_PRESENT: now also R403.2, TP403.1
- net RAIL_N12: now also C403.1, C405.1, C407.1, C409.1, D401.1 (K), R407.1, U40.11 (V-), U41.11 (V-)
- net RAIL_P12: now also C402.1, C404.1, C406.1, C408.1, D400.2 (A), U40.4 (V+), U41.4 (V+)
- net RETURN_FEED: now also R413.1, TP407.1
- net SHAPED_PRESENT: now also R412.1, TP406.1, U40.8 (OUT_C), U40.9 (IN_C-)
- new net ABS_CTRL_POS: R408.1, R409.1, U41.1 (OUT_A)
- new net ABS_CTRL_SUM: R406.2, R407.2, R408.2, U41.2 (IN_A-)
- new net ABS_GATE: D404.2 (A), Q40.2 (G), R411.2, TP405.1
- new net ABS_GATE_DRIVE: R410.1, R411.1, U41.7 (OUT_B)
- new net ABS_GATE_SUM: R409.2, R410.2, U41.6 (IN_B-)
- new net ADC_BUFFER: R415.1, U41.8 (OUT_C), U41.9 (IN_C-)
- new net GND: C400.2, C402.2, C403.2, C404.2, C405.2, C406.2, C407.2, C408.2, C409.2, D404.1 (K), J40.2 (TIP_NORMAL), J40.3 (SLEEVE), Q40.3 (S), R401.2, R402.2, U40.12 (IN_D+), U40.5 (IN_B+), U41.12 (IN_D+), U41.3 (IN_A+), U41.5 (IN_B+)
- new net INPUT_AC: C401.2, R402.1, U40.3 (IN_A+)
- new net INPUT_BUFFER: R403.1, R404.1, TP402.1, U40.1 (OUT_A), U40.2 (IN_A-)
- new net INPUT_PROTECTED: C400.1, C401.1, D400.1 (K), D401.2 (A), R400.2, R401.1, TP401.1
- new net INPUT_SPARE_OUT: U41.13 (IN_D-), U41.14 (OUT_D)
- new net INPUT_TIP: J40.1 (TIP), R400.1, TP400.1
- new net MEMORY_SUM: R412.2, R413.2, R414.2, U40.13 (IN_D-)
- new net MEMORY_SUM_OUT: R414.1, U40.14 (OUT_D), U41.10 (IN_C+)
- new net PRESSURE_OUT: C410.1, D402.1 (K), D403.2 (A), Q40.1 (D), R405.1, TP404.1, U40.10 (IN_C+), U40.7 (OUT_B)
- new net PRESSURE_SUM: C410.2, D402.2 (A), D403.1 (K), R404.2, R405.2, U40.6 (IN_B-)
Other:
- note added: "ADC_ANALOG_IN = -(SHAPED_PRESENT + RETURN_FEED), unity per input. The inverting sum restores the accepted feedback polarity from the inverting sheet-06 feed."
- note added: "DIRECT_PRESENT splits after protected AC-coupled unity buffering and before Pressure/Absence. SHAPED_PRESENT contains Pressure plus Return-derived Absence attenuation."
- note added: "J40/Q40/U40/U41 and diode footprints intentionally blank. JFET VGS(off), jack pin map, Pressure thresholds, Absence law, input surge behaviour and complete loop gain remain gates."
- note added: "No cable: J40 TIP normal contact grounds the input before protection. Plug insertion opens the normal contact and admits the external signal."
- note added: "SWITCHED INPUT • QUIET NO-CABLE STATE • DIRECT PRESENT • PRESSURE • ABSENCE • MEMORY SUM"
- note removed: "HIERARCHY / INTERFACE CAPTURE ONLY — CIRCUIT CONTENT NOT YET ACCEPTED"
- title: Memory Core Prototype A — INPUT / PRESSURE / ABSENCE -> Memory Core Prototype A — Input / Pressure / Absence

Commit message: Complete final integrated schematic review
Changed lines of the file:
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@@
 	)
 	(hierarchical_label "DIRECT_PRESENT"
-		(shape input)
+		(shape output)
 		(at 391.16 30.48 0.0000)
 		(effects
@@
 	)
 	(hierarchical_label "SHAPED_PRESENT"
-		(shape input)
+		(shape output)
 		(at 391.16 49.53 0.0000)
 		(effects
@@
 	)
 	(hierarchical_label "ADC_ANALOG_IN"
-		(shape input)
+		(shape output)
 		(at 391.16 68.58 0.0000)
 		(effects

Commit message: V5.4 — Verify input and output jack exact parts (#47)
Accept the WQP518MA/PJ398SM contact and PCB-footprint geometry, add the numeric project-local jack footprint, assign it to J40 and J70, preserve the blank project-symbol default, record the corrected 1.60 mm nut-only fit, and retain all PCB, panel and purchasing blocks.
Parts:
- J40: footprint (none) -> MerrinLab_PrototypeA:Jack_3.5mm_Thonkiconn_WQP518MA_Numeric
Changed lines of the file:
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@@
 			)
 		)
-		(property "Footprint" ""
+		(property "Footprint" "MerrinLab_PrototypeA:Jack_3.5mm_Thonkiconn_WQP518MA_Numeric"
 			(at 55.88 91.44 0.0000)
 			(effects
