File: hardware/memory-core-prototype-a/05_MEMORY_GHOST_WET.kicad_sch (KiCad schematic)
At the start: 1 part, among them J905 SHEET_INTERFACE_NOT_FITTED

Commit message: Capture ERC-validated Memory Ghost wet sheet
Parts:
- removed J905: SHEET_INTERFACE_NOT_FITTED, symbol Connector_Generic:Conn_01x08
- added C500, C504, C520: 10uF AC, symbol Device:C
- added C501, C505, C521: 1.2nF stability, Capacitor_SMD:C_0805_2012Metric, symbol Device:C
- added C502, C506, C522: 100nF control filter, Capacitor_SMD:C_0805_2012Metric, symbol Device:C
- added C503, C507, C523: 100pF I/V, Capacitor_SMD:C_0805_2012Metric, symbol Device:C
- added C510: 220pF sum bandwidth, Capacitor_SMD:C_0805_2012Metric, symbol Device:C
- added C530: 100nF + rail, Capacitor_SMD:C_0805_2012Metric, symbol Device:C
- added C531: 100nF - rail, Capacitor_SMD:C_0805_2012Metric, symbol Device:C
- added C532: 4.7uF + rail, Capacitor_SMD:C_0805_2012Metric, symbol Device:C
- added C533: 4.7uF - rail, Capacitor_SMD:C_0805_2012Metric, symbol Device:C
- added R500, R504, R520: 20k SSI input, Resistor_SMD:R_0805_2012Metric, symbol Device:R
- added R501, R505, R521: 220R stability, Resistor_SMD:R_0805_2012Metric, symbol Device:R
- added R502, R506, R522: 1k control isolate, Resistor_SMD:R_0805_2012Metric, symbol Device:R
- added R503, R507, R523: 20k I/V, Resistor_SMD:R_0805_2012Metric, symbol Device:R
- added R510: 40.2k 1% Memory sum, Resistor_SMD:R_0805_2012Metric, symbol Device:R
- added R511: 40.2k 1% Ghost sum, Resistor_SMD:R_0805_2012Metric, symbol Device:R
- added R512: 20k 1% half-sum feedback, Resistor_SMD:R_0805_2012Metric, symbol Device:R
- added R524: 47R output isolate, Resistor_SMD:R_0805_2012Metric, symbol Device:R
- added TP500: MEMORY_DAC, symbol Connector:TestPoint
- added TP501: MEMORY_VCA, symbol Connector:TestPoint
- added TP502: GHOST_DAC, symbol Connector:TestPoint
- added TP503: GHOST_VCA, symbol Connector:TestPoint
- added TP504: WET_SUM, symbol Connector:TestPoint
- added TP505: WET_MIX, symbol Connector:TestPoint
- added TP506: SSI_VC1, symbol Connector:TestPoint
- added TP507: SSI_VC2, symbol Connector:TestPoint
- added TP508: SSI_VC4, symbol Connector:TestPoint
- added U50: OPA1679 MEMORY/GHOST/WET, symbol MerrinLab_PrototypeA:OPA1679_PW_APPLICATION
- added U60: SSI2164, symbol MerrinLab_PrototypeA:SSI2164S_MULTI
Connections:
- net GHOST_DAC: now also C504.1, TP502.1
- net MEMORY_DAC: now also C500.1, TP500.1
- net RAIL_N12: now also C531.1, C533.1, U50.11 (V-)
- net RAIL_P12: now also C530.1, C532.1, U50.4 (V+)
- net VCA_GHOST_CTRL: now also R506.1
- net VCA_MEMORY_CTRL: now also R502.1
- net VCA_WET_CTRL: now also R522.1
- net WET_MIX: now also R524.2, TP505.1
- new net GHOST_VCA: C507.1, R507.1, R511.1, TP503.1, U50.7 (OUT_B)
- new net GHOST_VCA_AC: C504.2, R504.1
- new net GND: C501.2, C502.2, C505.2, C506.2, C521.2, C522.2, C530.2, C531.2, C532.2, C533.2, U50.10 (IN_C+), U50.12 (IN_D+), U50.3 (IN_A+), U50.5 (IN_B+)
- new net MEMORY_VCA: C503.1, R503.1, R510.1, TP501.1, U50.1 (OUT_A)
- new net MEMORY_VCA_AC: C500.2, R500.1
- new net SSI_IIN1: R500.2, R501.1, U60.2 (IIN1)
- new net SSI_IIN2: R504.2, R505.1, U60.7 (IIN2)
- new net SSI_IIN4: R520.2, R521.1, U60.10 (IIN4)
- new net SSI_IOUT1: C503.2, R503.2, U50.2 (IN_A-), U60.4 (IOUT1)
- new net SSI_IOUT2: C507.2, R507.2, U50.6 (IN_B-), U60.5 (IOUT2)
- new net SSI_IOUT4: C523.2, R523.2, U50.13 (IN_D-), U60.12 (IOUT4)
- new net SSI_STAB1: C501.1, R501.2
- new net SSI_STAB2: C505.1, R505.2
- new net SSI_STAB4: C521.1, R521.2
- new net SSI_VC1: C502.1, R502.2, TP506.1, U60.3 (VC1)
- new net SSI_VC2: C506.1, R506.2, TP507.1, U60.6 (VC2)
- new net SSI_VC4: C522.1, R522.2, TP508.1, U60.11 (VC4)
- new net WET_MASTER_AC: C520.2, R520.1
- new net WET_MASTER_OUT: C523.1, R523.1, R524.1, U50.14 (OUT_D)
- new net WET_SUM: C510.1, C520.1, R512.1, TP504.1, U50.8 (OUT_C)
- new net WET_SUM_NODE: C510.2, R510.2, R511.2, R512.2, U50.9 (IN_C-)
Other:
- note added: "BOUNDARY Memory, Ghost, wet-sum, SSI current nodes and controls remain local. Only WET_MIX crosses the sheet-05 hierarchy boundary."
- note added: "GHOST: pins 7 IIN2, 6 VC2, 5 IOUT2"
- note added: "MEM: pins 2 IIN1, 3 VC1, 4 IOUT1"
- note added: "SHARED DEVICE CONTRACT U60 unit 1 = Memory (2 IIN1, 3 VC1, 4 IOUT1). U60 unit 2 = Ghost (7 IIN2, 6 VC2, 5 IOUT2). U60 unit 4 = wet master (10 IIN4, 11 VC4, 12 IOUT4). U60 units 3 and 5 remain on sheet 06; no second SSI2164 is created."
- note added: "SSI2164 CH1 MEMORY • CH2 GHOST • EQUAL HALF-SUM • CH4 WET MASTER"
- note added: "WET SUM CONTRACT R510 = R511 = 40.2k; R512 = 20.0k. Each branch magnitude = 0.4975; two equal full-scale branches ~= 0.995 total. VCA controls are bounded and fail-safe-selected on sheet 08; sheet 05 adds isolation/filtering only."
- note added: "WET: pins 10 IIN4, 11 VC4, 12 IOUT4"
- note removed: "HIERARCHY / INTERFACE CAPTURE ONLY — CIRCUIT CONTENT NOT YET ACCEPTED"
- title: Memory Core Prototype A — MEMORY / GHOST / WET -> Memory Core Prototype A — Memory / Ghost / Wet

Commit message: Implement validated SSI2164 buffered control
Parts:
- added D500, D502, D504: BAT54-class upper clamp, symbol Device:D_Schottky
- added D501, D503, D505: BAT54-class lower clamp, symbol Device:D_Schottky
- added R525, R526, R527: 20R buffer isolate, Resistor_SMD:R_0805_2012Metric, symbol Device:R
- added U63: OPA4196 CONTROL BUFFER, symbol MerrinLab_PrototypeA:OPA4196_PW_MULTI
- R502, R506, R522: value 1k control isolate -> 1k pre-buffer filter
Connections:
- net GND: now also D501.2 (A), D503.2 (A), D505.2 (A)
- net SSI_VC1: now also D500.2 (A), D501.1 (K), R525.2; no longer C502.1, R502.2
- net SSI_VC2: now also D502.2 (A), D503.1 (K), R526.2; no longer C506.1, R506.2
- net SSI_VC4: now also D504.2 (A), D505.1 (K), R527.2; no longer C522.1, R522.2
- new net GHOST_CTRL_BUFFER_IN: C506.1, R506.2, U63.5 (+IN_B)
- new net GHOST_CTRL_BUFFER_OUT: R526.1, U63.6 (-IN_B), U63.7 (OUT_B)
- new net MEM_CTRL_BUFFER_IN: C502.1, R502.2, U63.3 (+IN_A)
- new net MEM_CTRL_BUFFER_OUT: R525.1, U63.1 (OUT_A), U63.2 (-IN_A)
- new net RAIL_3V3: D500.1 (K), D502.1 (K), D504.1 (K)
- new net WET_CTRL_BUFFER_IN: C522.1, R522.2, U63.12 (+IN_D)
- new net WET_CTRL_BUFFER_OUT: R527.1, U63.13 (-IN_D), U63.14 (OUT_D)
Other:
- note added: "SHARED DEVICE CONTRACT U60 unit 1 = Memory (2 IIN1, 3 VC1, 4 IOUT1). U60 unit 2 = Ghost (7 IIN2, 6 VC2, 5 IOUT2). U60 unit 4 = wet master (10 IIN4, 11 VC4, 12 IOUT4). U60 units 3 and 5 remain on sheet 06; no second SSI2164 is created. U63 OPA4196 units 1/2/4 buffer Memory/Ghost/Wet; units 3/5 remain on sheet 06."
- note removed: "SHARED DEVICE CONTRACT U60 unit 1 = Memory (2 IIN1, 3 VC1, 4 IOUT1). U60 unit 2 = Ghost (7 IIN2, 6 VC2, 5 IOUT2). U60 unit 4 = wet master (10 IIN4, 11 VC4, 12 IOUT4). U60 units 3 and 5 remain on sheet 06; no second SSI2164 is created."
